File: sch/KiCAD/cellular-polymaton.sch (KiCad schematic (older format))
At the start: 26 parts, among them P1 CONN_5X2, P2 CONN_5X2, P3 CONN_5X2, P4 CONN_5X2, P5 CONN_5X2, U1 74HC595, U2 74HC595, U3 74HC595, U4 74HC595, U5 74HC595, U6 LM323T

Commit message: recreated board file and made config.g for Automaton 0x01
Parts:
- gave numbers to parts that had none: 15
Changed lines of the file:
@@
-EESchema Schematic File Version 2  date Wed 29 Feb 2012 04:03:13 PM PST
+EESchema Schematic File Version 2  date Wed 07 Mar 2012 01:31:47 PM PST
 LIBS:power
 LIBS:device
@@
 LIBS:valves
 LIBS:myparts
-EELAYER 43  0
+LIBS:cellular-polymaton-cache
+EELAYER 25  0
 EELAYER END
 $Descr A4 11700 8267
@@
 Sheet 1 1
 Title ""
-Date "1 mar 2012"
+Date "7 mar 2012"
 Rev ""
 Comp ""
@@
 5V
 $Comp
-L GND #PWR?
+L GND #PWR1
 U 1 1 4F4EB853
 P 1800 800
-F 0 "#PWR?" H 1800 800 30  0001 C CNN
+F 0 "#PWR1" H 1800 800 30  0001 C CNN
 F 1 "GND" H 1800 730 30  0001 C CNN
 	1    1800 800
@@
 $EndComp
 $Comp
-L GND #PWR?
+L GND #PWR2
 U 1 1 4F4EB6FA
 P 3350 2600
-F 0 "#PWR?" H 3350 2600 30  0001 C CNN
+F 0 "#PWR2" H 3350 2600 30  0001 C CNN
 F 1 "GND" H 3350 2530 30  0001 C CNN
 	1    3350 2600
@@
 $EndComp
 $Comp
-L CONN_2 P?
+L CONN_2 P6
 U 1 1 4F4EB608
 P 4500 7250
-F 0 "P?" V 4450 7250 40  0000 C CNN
+F 0 "P6" V 4450 7250 40  0000 C CNN
 F 1 "CONN_2" V 4550 7250 40  0000 C CNN
 	1    4500 7250
@@
 $EndComp
 $Comp
-L SWITCH_INV SW?
+L SWITCH_INV SW1
 U 1 1 4F4EB5A2
 P 2200 1300
-F 0 "SW?" H 2000 1450 50  0000 C CNN
+F 0 "SW1" H 2000 1450 50  0000 C CNN
 F 1 "SWITCH_INV" H 2050 1150 50  0000 C CNN
 	1    2200 1300
@@
 $EndComp
 $Comp
-L R R?
+L R R1
 U 1 1 4F4EB56D
 P 4400 1650
-F 0 "R?" V 4480 1650 50  0000 C CNN
+F 0 "R1" V 4480 1650 50  0000 C CNN
 F 1 "R" V 4400 1650 50  0000 C CNN
 	1    4400 1650
@@
 $EndComp
 $Comp
-L R R?
+L R R2
 U 1 1 4F4EB521
 P 5800 4000
-F 0 "R?" V 5880 4000 50  0000 C CNN
+F 0 "R2" V 5880 4000 50  0000 C CNN
 F 1 "R" V 5800 4000 50  0000 C CNN
 	1    5800 4000
@@
 $EndComp
 $Comp
-L CONN_3 K?
+L CONN_3 K1
 U 1 1 4F4EB513
 P 950 1200
-F 0 "K?" V 900 1200 50  0000 C CNN
+F 0 "K1" V 900 1200 50  0000 C CNN
 F 1 "CONN_3" V 1000 1200 40  0000 C CNN
 	1    950  1200
@@
 $EndComp
 $Comp
-L LED D?
+L LED D2
 U 1 1 4F4EB4F5
 P 4400 2100
-F 0 "D?" H 4400 2200 50  0000 C CNN
+F 0 "D2" H 4400 2200 50  0000 C CNN
 F 1 "LED" H 4400 2000 50  0000 C CNN
 	1    4400 2100
@@
 $EndComp
 $Comp
-L C C?
+L C C6
 U 1 1 4F4EB4EF
 P 2000 7300
-F 0 "C?" H 2050 7400 50  0000 L CNN
+F 0 "C6" H 2050 7400 50  0000 L CNN
 F 1 "C" H 2050 7200 50  0000 L CNN
 	1    2000 7300
@@
 $EndComp
 $Comp
-L C C?
+L C C4
 U 1 1 4F4EB4ED
 P 1400 7250
-F 0 "C?" H 1450 7350 50  0000 L CNN
+F 0 "C4" H 1450 7350 50  0000 L CNN
 F 1 "C" H 1450 7150 50  0000 L CNN
 	1    1400 7250
@@
 $EndComp
 $Comp
-L C C?
+L C C2
 U 1 1 4F4EB4EB
 P 950 7250
-F 0 "C?" H 1000 7350 50  0000 L CNN
+F 0 "C2" H 1000 7350 50  0000 L CNN
 F 1 "C" H 1000 7150 50  0000 L CNN
 	1    950  7250
@@
 $EndComp
 $Comp
-L C C?
+L C C5
 U 1 1 4F4EB4E9
 P 1900 6600
-F 0 "C?" H 1950 6700 50  0000 L CNN
+F 0 "C5" H 1950 6700 50  0000 L CNN
 F 1 "C" H 1950 6500 50  0000 L CNN
 	1    1900 6600
@@
 $EndComp
 $Comp
-L C C?
+L C C3
 U 1 1 4F4EB4E7
 P 1350 6700
-F 0 "C?" H 1400 6800 50  0000 L CNN
+F 0 "C3" H 1400 6800 50  0000 L CNN
 F 1 "C" H 1400 6600 50  0000 L CNN
 	1    1350 6700
@@
 $EndComp
 $Comp
-L C C?
+L C C1
 U 1 1 4F4EB4DE
 P 900 6700
-F 0 "C?" H 950 6800 50  0000 L CNN
+F 0 "C1" H 950 6800 50  0000 L CNN
 F 1 "C" H 950 6600 50  0000 L CNN
 	1    900  6700
@@
 $EndComp
 $Comp
-L DIODE D?
+L DIODE D1
 U 1 1 4F4EB43E
 P 1500 1300
-F 0 "D?" H 1500 1400 40  0000 C CNN
+F 0 "D1" H 1500 1400 40  0000 C CNN
 F 1 "DIODE" H 1500 1200 40  0000 C CNN
 	1    1500 1300
@@
 $EndComp
 $Comp
-L CP1 C?
+L CP1 C8
 U 1 1 4F4EB43A
 P 4000 1600
-F 0 "C?" H 4050 1700 50  0000 L CNN
+F 0 "C8" H 4050 1700 50  0000 L CNN
 F 1 "CP1" H 4050 1500 50  0000 L CNN
 	1    4000 1600
@@
 $EndComp
 $Comp
-L CP1 C?
+L CP1 C7
 U 1 1 4F4EB437
 P 2700 1600
-F 0 "C?" H 2750 1700 50  0000 L CNN
+F 0 "C7" H 2750 1700 50  0000 L CNN
 F 1 "CP1" H 2750 1500 50  0000 L CNN
 	1    2700 1600
